File: kicad/kicad/delay-generator.kicad_pcb (KiCad board)
At the start: 2 copper layers, 114.3 x 63.5 mm, 24 parts, among them U1 L7805, U2 74LS121, U3 74LS121

Commit message: plumbing
Parts:
- moved R2 16.3 mm to (147.3, 78.7)
- moved R1 16.3 mm to (129.5, 73.7)
- moved TP_5V1 16.3 mm to (68.6, 78.7)
- moved U3 16.3 mm to (137.2, 73.7)
- moved C2 16.3 mm to (96.5, 45.7)
- moved J_POWER1 16.3 mm to (83.8, 45.7)
- moved REF** 16.3 mm to (68.6, 45.7)
- moved R_DELAY1 16.3 mm to (109.2, 55.9)
- moved C1 16.3 mm to (86.4, 58.4)
- moved C3 16.3 mm to (68.6, 58.4)
- moved J_INPUT1 16.3 mm to (91.4, 99.1)
- moved REF** 16.3 mm to (68.6, 99.1)
- moved TP_COM1 16.3 mm to (68.6, 71.1)
- moved U1 16.3 mm to (81.3, 71.1)
- moved U2 16.3 mm to (101.6, 73.7)
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Other:
- board text added: "DELAY GENERATOR BLAISE THOMPSON MARCH 2022"
- board text removed: "DELAY GENERATOR BLAISE THOMPSON APRIL 2019"

Commit message: pcb training
Other:
- board text added: "DELAY GENERATOR BLAISE THOMPSON MARCH 2023"
- board text removed: "DELAY GENERATOR BLAISE THOMPSON MARCH 2022"
