File: kicad/kicad/delay-generator.kicad_sch (KiCad schematic)
At the start: 20 parts, among them U1 L7805, U2 74LS121, U3 74LS121

Commit message: plumbing
Parts:
- removed C1: 100uF, Capacitor_THT:CP_Radial_D7.5mm_P2.50mm, symbol Device:CP1
- removed C2: 330nF, Capacitor_THT:CP_Radial_D7.5mm_P2.50mm, symbol Device:CP1
- removed C3: 100nF, Capacitor_THT:CP_Radial_D7.5mm_P2.50mm, symbol Device:CP1
- added C1: 100u, Capacitor_THT:CP_Radial_D7.5mm_P2.50mm, symbol Device:C_Polarized_US
- added C2: 330n, Capacitor_THT:CP_Radial_D7.5mm_P2.50mm, symbol Device:C_Polarized_US
- added C3: 100n, Capacitor_THT:CP_Radial_D7.5mm_P2.50mm, symbol Device:C_Polarized_US
- C4: footprint Capacitor_THT:CP_Radial_D7.5mm_P2.50mm -> Capacitor_THT:C_Disc_D7.5mm_W4.4mm_P5.00mm
Connections:
- net +5V: now also C3.1
- net GND: now also C1.2, C2.2, C3.2
- net at J_POWER1.2 (Pin_2), U1.1 (IN): now also C1.1, C2.1
Changed lines of the file:
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@@
   (title_block
     (title "Delay Generator")
-    (date "2019-04-17")
+    (date "2022-03-21")
     (rev "A")
     (company "UW-Madison")
     (comment 1 "Department of Chemistry")
+    (comment 2 "Instrument Shop")
+    (comment 3 "Blaise Thompson")
+    (comment 4 "blaise.thompson@wisc.edu")
   )
   (junction (at 36.83 120.65) (diameter 0) (color 0 0 0 0)
   )
+  (junction (at 232.41 96.52) (diameter 0) (color 0 0 0 0)
+  )
+  (junction (at 109.22 91.44) (diameter 0) (color 0 0 0 0)
+  )
+  (junction (at 44.45 95.25) (diameter 0) (color 0 0 0 0)
+  )
   (junction (at 36.83 95.25) (diameter 0) (color 0 0 0 0)
-  )
-  (junction (at 232.41 96.52) (diameter 0) (color 0 0 0 0)
-  )
-  (junction (at 109.22 91.44) (diameter 0) (color 0 0 0 0)
-  )
-  (junction (at 44.45 95.25) (diameter 0) (color 0 0 0 0)
   )
   (junction (at 69.85 95.25) (diameter 0) (color 0 0 0 0)
@@
     (stroke (width 0) (type default) (color 0 0 0 0))
   )
+  (wire (pts (xy 119.38 91.44) (xy 109.22 91.44))
+    (stroke (width 0) (type default) (color 0 0 0 0))
+  )
+  (wire (pts (xy 201.93 104.14) (xy 190.5 104.14))
+    (stroke (width 0) (type default) (color 0 0 0 0))
+  )
+  (wire (pts (xy 69.85 104.14) (xy 72.39 104.14))
+    (stroke (width 0) (type default) (color 0 0 0 0))
+  )
+  (wire (pts (xy 69.85 104.14) (xy 69.85 109.22))
+    (stroke (width 0) (type default) (color 0 0 0 0))
+  )
+  (wire (pts (xy 165.1 96.52) (xy 165.1 106.68))
+    (stroke (width 0) (type default) (color 0 0 0 0))
+  )
+  (wire (pts (xy 190.5 104.14) (xy 190.5 111.76))
+    (stroke (width 0) (type default) (color 0 0 0 0))
+  )
+  (wire (pts (xy 116.84 104.14) (xy 116.84 106.68))
+    (stroke (width 0) (type default) (color 0 0 0 0))
+  )
+  (wire (pts (xy 109.22 87.63) (xy 109.22 91.44))
+    (stroke (width 0) (type default) (color 0 0 0 0))
+  )
+  (wire (pts (xy 64.77 95.25) (xy 69.85 95.25))
+    (stroke (width 0) (type default) (color 0 0 0 0))
+  )
+  (wire (pts (xy 57.15 120.65) (xy 57.15 109.22))
+    (stroke (width 0) (type default) (color 0 0 0 0))
+  )
+  (wire (pts (xy 57.15 102.87) (xy 57.15 109.22))
+    (stroke (width 0) (type default) (color 0 0 0 0))
+  )
   (wire (pts (xy 36.83 95.25) (xy 36.83 120.65))
-    (stroke (width 0) (type default) (color 0 0 0 0))
-  )
-  (wire (pts (xy 119.38 91.44) (xy 109.22 91.44))
-    (stroke (width 0) (type default) (color 0 0 0 0))
-  )
-  (wire (pts (xy 201.93 104.14) (xy 190.5 104.14))
-    (stroke (width 0) (type default) (color 0 0 0 0))
-  )
-  (wire (pts (xy 69.85 104.14) (xy 72.39 104.14))
-    (stroke (width 0) (type default) (color 0 0 0 0))
-  )
-  (wire (pts (xy 69.85 104.14) (xy 69.85 109.22))
-    (stroke (width 0) (type default) (color 0 0 0 0))
-  )
-  (wire (pts (xy 165.1 96.52) (xy 165.1 106.68))
-    (stroke (width 0) (type default) (color 0 0 0 0))
-  )
-  (wire (pts (xy 190.5 104.14) (xy 190.5 111.76))
-    (stroke (width 0) (type default) (color 0 0 0 0))
-  )
-  (wire (pts (xy 116.84 104.14) (xy 116.84 106.68))
-    (stroke (width 0) (type default) (color 0 0 0 0))
-  )
-  (wire (pts (xy 109.22 87.63) (xy 109.22 91.44))
-    (stroke (width 0) (type default) (color 0 0 0 0))
-  )
-  (wire (pts (xy 64.77 95.25) (xy 69.85 95.25))
-    (stroke (width 0) (type default) (color 0 0 0 0))
-  )
-  (wire (pts (xy 57.15 120.65) (xy 57.15 109.22))
-    (stroke (width 0) (type default) (color 0 0 0 0))
-  )
-  (wire (pts (xy 57.15 102.87) (xy 57.15 109.22))
     (stroke (width 0) (type default) (color 0 0 0 0))
   )
@@
     (pin "2")
   )
-  (symbol (lib_id "Device:CP1") (at 63.5 109.22 270) (unit 1)
-    (in_bom yes) (on_board yes)
-    (property "Reference" "C3" (id 0) (at 63.5 102.8192 90))
-    (property "Value" "100nF" (id 1) (at 63.5 105.1306 90))
-    (property "Footprint" "Capacitor_THT:CP_Radial_D7.5mm_P2.50mm" (id 2) (at 63.5 109.22 0)
-      (effects (font (size 1.27 1.27)) hide)
-    )
-    (property "Datasheet" "~" (id 3) (at 63.5 109.22 0)
-      (effects (font (size 1.27 1.27)) hide)
-    )
-    (pin "1")
-    (pin "2")
-  )
-  (symbol (lib_id "Device:CP1") (at 50.8 109.22 90) (unit 1)
-    (in_bom yes) (on_board yes)
-    (property "Reference" "C2" (id 0) (at 50.8 102.8192 90))
-    (property "Value" "330nF" (id 1) (at 50.8 105.1306 90))
-    (property "Footprint" "Capacitor_THT:CP_Radial_D7.5mm_P2.50mm" (id 2) (at 50.8 109.22 0)
-      (effects (font (size 1.27 1.27)) hide)
-    )
-    (property "Datasheet" "~" (id 3) (at 50.8 109.22 0)
-      (effects (font (size 1.27 1.27)) hide)
-    )
-    (pin "1")
-    (pin "2")
-  )
   (symbol (lib_id "power:+5V") (at 72.39 104.14 0) (unit 1)
     (in_bom yes) (on_board yes)
@@
       (effects (font (size 1.27 1.27)) (justify left))
     )
-    (property "Footprint" "Capacitor_THT:CP_Radial_D7.5mm_P2.50mm" (id 2) (at 108.2548 91.44 0)
+    (property "Footprint" "Capacitor_THT:C_Disc_D7.5mm_W4.4mm_P5.00mm" (id 2) (at 108.2548 91.44 0)
       (effects (font (size 1.27 1.27)) hide)
     )
@@
     (pin "1")
   )
-  (symbol (lib_id "Device:CP1") (at 40.64 95.25 270) (unit 1)
-    (in_bom yes) (on_board yes)
-    (property "Reference" "C1" (id 0) (at 40.64 101.6508 90))
-    (property "Value" "100uF" (id 1) (at 40.64 99.3394 90))
+  (symbol (lib_id "Device:C_Polarized_US") (at 63.5 109.22 270) (unit 1)
+    (in_bom yes) (on_board yes) (fields_autoplaced)
+    (property "Reference" "C3" (id 0) (at 64.135 101.6 90))
+    (property "Value" "100n" (id 1) (at 64.135 104.14 90))
+    (property "Footprint" "Capacitor_THT:CP_Radial_D7.5mm_P2.50mm" (id 2) (at 63.5 109.22 0)
+      (effects (font (size 1.27 1.27)) hide)
+    )
+    (property "Datasheet" "~" (id 3) (at 63.5 109.22 0)
+      (effects (font (size 1.27 1.27)) hide)
+    )
+    (pin "1")
+    (pin "2")
+  )
+  (symbol (lib_id "Device:C_Polarized_US") (at 50.8 109.22 90) (unit 1)
+    (in_bom yes) (on_board yes) (fields_autoplaced)
+    (property "Reference" "C2" (id 0) (at 50.165 101.6 90))
+    (property "Value" "330n" (id 1) (at 50.165 104.14 90))
+    (property "Footprint" "Capacitor_THT:CP_Radial_D7.5mm_P2.50mm" (id 2) (at 50.8 109.22 0)
+      (effects (font (size 1.27 1.27)) hide)
+    )
+    (property "Datasheet" "~" (id 3) (at 50.8 109.22 0)
+      (effects (font (size 1.27 1.27)) hide)
+    )
+    (pin "1")
+    (pin "2")
+  )
+  (symbol (lib_id "Device:C_Polarized_US") (at 40.64 95.25 270) (unit 1)
+    (in_bom yes) (on_board yes) (fields_autoplaced)
+    (property "Reference" "C1" (id 0) (at 41.275 87.63 90))
+    (property "Value" "100u" (id 1) (at 41.275 90.17 90))
     (property "Footprint" "Capacitor_THT:CP_Radial_D7.5mm_P2.50mm" (id 2) (at 40.64 95.25 0)
       (effects (font (size 1.27 1.27)) hide)
@@
       (reference "#PWR0111") (unit 1) (value "GND") (footprint "")
     )
-    (path "/00000000-0000-0000-0000-00005cbc8be7"
-      (reference "C1") (unit 1) (value "100uF") (footprint "Capacitor_THT:CP_Radial_D7.5mm_P2.50mm")
-    )
-    (path "/00000000-0000-0000-0000-00005cb56490"
-      (reference "C2") (unit 1) (value "330nF") (footprint "Capacitor_THT:CP_Radial_D7.5mm_P2.50mm")
-    )
-    (path "/00000000-0000-0000-0000-00005cb55e28"
-      (reference "C3") (unit 1) (value "100nF") (footprint "Capacitor_THT:CP_Radial_D7.5mm_P2.50mm")
+    (path "/e325a134-36dc-4151-9d17-8bf13dc78564"
+      (reference "C1") (unit 1) (value "100u") (footprint "Capacitor_THT:CP_Radial_D7.5mm_P2.50mm")
+    )
+    (path "/b2364ccc-d560-471e-96fb-ac59e9de768a"
+      (reference "C2") (unit 1) (value "330n") (footprint "Capacitor_THT:CP_Radial_D7.5mm_P2.50mm")
+    )
+    (path "/15a65612-f6a1-48be-8425-8f5afb06c4fd"
+      (reference "C3") (unit 1) (value "100n") (footprint "Capacitor_THT:CP_Radial_D7.5mm_P2.50mm")
     )
     (path "/00000000-0000-0000-0000-00005cb68d4c"
-      (reference "C4") (unit 1) (value "1uF") (footprint "Capacitor_THT:CP_Radial_D7.5mm_P2.50mm")
+      (reference "C4") (unit 1) (value "1uF") (footprint "Capacitor_THT:C_Disc_D7.5mm_W4.4mm_P5.00mm")
     )
     (path "/00000000-0000-0000-0000-00005cb8cdb6"
